File: uMyo_v3_1/uMyo_v3_1.kicad_pcb (KiCad board)
At the start: 2 copper layers, 47.1 x 28 mm, 53 parts, among them J1 Conn_01x01_Male, J2 Conn_01x01_Male, J4 Conn_01x01_Male, J5 Conn_01x01_Male, J6 Conn_01x02_Female, J7 Conn_01x02_Female, SW1 SW_Push, U1 AD8293G80ARJZ-R2, U2 nRF52810-QFxx, U3 XC6206P332MR_SOT23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

Commit message: Edit Back Silkcreen
- Add Cura Logo
- Add Batch Number
- Add Season where batch was printed
- Add my name and ID
Parts:
- added G***: LOGO, LOGO, B.Cu at (123.0, 95.8)
Other:
- board text added: "B01 | SP26 ZSE • 61-3864"
