File: uMyo_v3_1/uMyo_v3_1.kicad_pcb (KiCad board)
At the start: 2 copper layers, 47.1 x 28 mm, 54 parts, among them J1 Conn_01x01_Male, J2 Conn_01x01_Male, J4 Conn_01x01_Male, J5 Conn_01x01_Male, J6 Conn_01x02_Female, J7 Conn_01x02_Female, SW1 SW_Push, U1 AD8293G80ARJZ-R2, U2 nRF52810-QFxx, U3 XC6206P332MR_SOT23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

Commit message: Add JLCPCB constraints and run DRC
Other:
- copper layers 2 -> 4
Changed lines of the file:
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@@
 	(generator_version "9.0")
 	(general
-		(thickness 1.6)
+		(thickness 1.600198)
 		(legacy_teardrops no)
 	)
@@
 	(layers
 		(0 "F.Cu" signal)
+		(4 "In1.Cu" signal)
+		(6 "In2.Cu" signal)
 		(2 "B.Cu" signal)
-		(9 "F.Adhes" user "F.Adhesive")
-		(11 "B.Adhes" user "B.Adhesive")
 		(13 "F.Paste" user)
 		(15 "B.Paste" user)
@@
 		(1 "F.Mask" user)
 		(3 "B.Mask" user)
-		(17 "Dwgs.User" user "User.Drawings")
-		(19 "Cmts.User" user "User.Comments")
-		(21 "Eco1.User" user "User.Eco1")
-		(23 "Eco2.User" user "User.Eco2")
 		(25 "Edge.Cuts" user)
 		(27 "Margin" user)
@@
 		(29 "B.CrtYd" user "B.Courtyard")
 		(35 "F.Fab" user)
-		(33 "B.Fab" user)
 	)
 	(setup
@@
 			(layer "F.SilkS"
 				(type "Top Silk Screen")
-				(color "Black")
 			)
 			(layer "F.Paste"
@@
 			(layer "F.Mask"
 				(type "Top Solder Mask")
-				(color "#9E6B09D4")
 				(thickness 0.01)
 			)
@@
 			(layer "dielectric 1"
 				(type "core")
-				(thickness 1.51)
+				(thickness 0.480066)
+				(material "FR4")
+				(epsilon_r 4.5)
+				(loss_tangent 0.02)
+			)
+			(layer "In1.Cu"
+				(type "copper")
+				(thickness 0.035)
+			)
+			(layer "dielectric 2"
+				(type "prepreg")
+				(thickness 0.480066)
+				(material "FR4")
+				(epsilon_r 4.5)
+				(loss_tangent 0.02)
+			)
+			(layer "In2.Cu"
+				(type "copper")
+				(thickness 0.035)
+			)
+			(layer "dielectric 3"
+				(type "core")
+				(thickness 0.480066)
 				(material "FR4")
 				(epsilon_r 4.5)
@@
 			(layer "B.Mask"
 				(type "Bottom Solder Mask")
-				(color "#9E6B09D4")
 				(thickness 0.01)
 			)
@@
 			(layer "B.SilkS"
 				(type "Bottom Silk Screen")
-				(color "Black")
 			)
 			(copper_finish "None")
@@
 		)
 		(pad_to_mask_clearance 0)
+		(solder_mask_min_width 0.12)
 		(allow_soldermask_bridges_in_footprints no)
 		(tenting front back)
@@
 		(layer "F.SilkS")
 	)
-	(gr_circle
-		(center 141.2 98)
-		(end 144.7 98)
-		(stroke
-			(width 0.15)
-			(type solid)
-		)
-		(fill no)
-		(layer "Dwgs.User")
-	)
 	(gr_line
